File: Hardware/P1-lezer.kicad_pcb (KiCad board)
At the start: 2 copper layers, 70 x 30 mm, 13 parts, among them J1 RJ12, M2.5 MountingHole_2.7mm_M2.5_ISO73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, Q1 BC547, U1 WeMos_D1_mini, U2 TIL111

Commit message: Added github-URL
Other:
- board text added: "https://github.com/StoffelNL/P1-Lezer"
Changed lines of the file:
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@@
 		(layer "Edge.Cuts")
+	)
+	(gr_text "https://github.com/StoffelNL/P1-Lezer"
+		(at 103 96.2 0)
+		(layer "B.SilkS")
+		(effects
+			(font
+				(size 1 1)
+				(thickness 0.153)
+			)
+			(justify left bottom mirror)
+		)
 	)
 	(gr_text "P1-Lezer © 2024 StoffelNL"
